File: telemetry_station/station.kicad_pcb (KiCad board)
At the start: 2 copper layers, 50 x 53.8 mm, 24 parts, among them J1 2.4Ghz, U11 SX1280IMLTRT, Y2 52Mhz

Commit message: Station schematic
Routing:
- net GND: track 0.00 -> 5.32 mm, vias 0 -> 31
- added copper zone on In1.Cu, net GND
- added copper zone on In2.Cu, net VCC
Other:
- copper layers 2 -> 4
