File: Microcontroler_2026_2027/Alimentation.kicad_sch (KiCad schematic)
At the start: 25 parts, among them J5 Screw_Terminal_01x04, Q1 AO3401A, U5 LMR33630ADDA, U6 TLV75533PDBV

Commit message: updated components footprints
Parts:
- renumbered C13 to C46, C14 to C47, C15 to C48, C16 to C49, C18 to C50, C20 to C51, C21 to C52, C22 to C53, C17 to C54, C19 to C55, D2 to D5, FB1 to FB2, J5 to J10, L1 to L5, Q1 to Q3, R2 to R16, R4 to R17, R6 to R18, R7 to R19, TP1 to TP13, TP3 to TP14, TP2 to TP15, TP4 to TP16, U5 to U11, U6 to U12
