File: Microcontroler_2026_2027/Secondarie_Controler.kicad_sch (KiCad schematic)
At the start: 39 parts, among them J10 APPS, J13 TC2030, J7 Screw_Terminal_01x04, J8 Brake_Sensor, Q3 AO3400A, SW1 SW_Push, U12 CR2013-MI2120, U13 TLV75533PDBV, U7 STM32G474RETx, U9 SN65HVD230

Commit message: Branch initial commit / TC2030 wired
Parts:
- removed J13: TC2030, Connector:Tag-Connect_TC2030-IDC-NL_2x03_P1.27mm_Vertical, symbol Connector:TC2030
- added J3: ST-LINK TC2030, Connector:Tag-Connect_TC2030-IDC-FP_2x03_P1.27mm_Vertical, symbol Connector:Conn_ARM_SWD_TagConnect_TC2030
- added R20: 10k, Resistor_SMD:R_1206_3216Metric, symbol Device:R_Small
Connections:
- net GND: now also J3.5 (GND)
- net VCC: now also J3.1 (VCC), R20.1
- net SWDIO: now reaches U7.49 (PA13)
- net SWDIO: now also J3.2 (SWDIO)
- net SWCLK: now reaches U7.50 (PA14)
- net SWCLK: now also J3.4 (SWCLK)
- net SWO: now reaches U7.56 (PB3)
- net SWO: now also J3.6 (SWO)
- net NRST: now reaches U7.7 (PG10)
- net NRST: now also J3.3 (~{RESET}), R20.2
- net RESET: no longer names the net of U7.22 (PC4)
- no-connect marks 35 -> 32
Other:
- note removed: "A FINIR"

Commit message: Added telemetry station schematic and wired SPI to the main controller
Parts:
- added Y4: 8Mhz, Oscillator:Oscillator_SMD_Abracon_ASCO-4Pin_1.6x1.2mm, symbol Oscillator:ASCO
Connections:
- net +12V is gone; now on net +5V: BZ1.1 (+), J7.3 (Pin_3)
- net +3.3V: now also Y4.1 (Tri-State), Y4.4 (VDD)
- net GND: now also Y4.2 (GND)
- net OSC_IN: now reaches U7.5 (PF0)
- net OSC_IN: now also Y4.3 (OUT)
- no-connect marks 32 -> 31
Other:
- note added: "8Mhz Oscillator"
- moved on the sheet: R20

Commit message: updated components footprints
Parts:
- renumbered C23 to C33, C52 to C34, C24 to C35, C53 to C36, C26 to C37, C28 to C38, C30 to C39, C31 to C40, C32 to C41, C34 to C42, C35 to C43, C37 to C44, C41 to C45, J3 to J6, J10 to J9, Q3 to Q2, R15 to R11, R16 to R12, R17 to R13, R18 to R14, R19 to R15, R20 to R7, TP9 to TP10, TP12 to TP11, TP13 to TP12, TP19 to TP9, U9 to U10, U13 to U7, U7 to U8, U12 to U9, Y4 to Y3
